File: ITR-1/ITR-1.sch (KiCad schematic (older format))
At the start: 44 parts, among them K1 Кнопка_KLS7-TS5401-1.35-250-T, X1 отверстие_под_пайку, X2 отверстие_под_пайку

Commit message: подготовлена трассировка +PNG +STP, требуется контрольная проверка
Parts:
- removed HL1: Светодиод_сдвоенный_KPB-3025SURKCGKC, N_VD_HL:Светодиод_SMD_m3025, symbol elements_2020:Светодиод_сдвоенный_KPB-3025SURKCGKC
- removed R16: Резистор_0,065Вт, N_RLC:Резистор_SMD_0603_0,065_Вт, symbol elements:Резистор_0,065Вт
- added D1: LOGO, N_ICO:ni_10x10, symbol elements:LOGO
- added D2: LOGO, N_ICO:VLAD_10x10, symbol elements:LOGO
- added HL1: Светодиод, N_VD_HL:Светодиод_SMD_IEC_0603, symbol BIG_schemes:Светодиод
Connections:
- net LED.RED is gone; now on net CHARGE.MODE: A1.31 (IO19)
- net AN.2V5.REF: now also A1.24 (IO2); no longer A1.5 (SENSOR_VN)
- net AN.BAT.MEASURE: now also A1.26 (IO4); no longer A1.7 (IO35)
- net BUTT.TURN: now also A1.28 (IO17); no longer A1.11 (IO26)
- net CHARGE.MODE: no longer A1.13 (IO14)
- net GND: now also HL1.K
- net SELF.TURN: now also A1.29 (IO5); no longer A1.9 (IO33)
- net LED: now reaches A1.30 (IO18)
- net LED: now also R17.2
- net at R17.1: now also HL1.A
- removed net LED.GREEN: A1.29 (IO5), R17.2
- no-connect marks 9 -> 3
Other:
- moved on the sheet: R17
Changed lines of the file:
@@
 $EndComp
 $Comp
-L elements_2020:Светодиод_сдвоенный_KPB-3025SURKCGKC HL1
-U 1 1 613366EC
-P 8000 9250
-F 0 "HL1" H 8150 9450 60  0000 C CNN
-F 1 "Светодиод_сдвоенный_KPB-3025SURKCGKC" H 8150 9489 60  0001 C CNN
-F 2 "N_VD_HL:Светодиод_SMD_m3025" H 8300 8750 60  0001 C CNN
-F 3 "" H 8300 8750 60  0001 C CNN
-	1    8000 9250
-	1    0    0    -1
-$EndComp
-$Comp
 L elements:стабилизатор_нерегулируемый_LM1117S33-SOT223 G1
 U 1 1 6133BBFC
@@
 Text Label 6275 8500 2    50   ~ 0
 GND
-Text Label 1750 10300 0    50   ~ 0
+Text Label 6750 9550 2    50   ~ 0
 CHARGE.MODE
-Text Label 1750 9700 0    50   ~ 0
-SELF.TURN
-Text Label 1750 10000 0    50   ~ 0
+Text Label 6750 10000 2    50   ~ 0
 BUTT.TURN
-Wire Wire Line
-	2500 9100 1750 9100
-Wire Wire Line
-	1750 9400 2500 9400
-NoConn ~ 2500 8950
 Text Label 2125 8800 0    50   ~ 0
 RESET
@@
 	6625 8950 5950 8950
 Wire Wire Line
-	1750 9700 2500 9700
-Wire Wire Line
-	1750 10000 2500 10000
-Wire Wire Line
-	1750 10300 2500 10300
-NoConn ~ 2500 9550
-NoConn ~ 2500 9850
-NoConn ~ 2500 10150
+	6750 9550 5950 9550
 Text Label 6250 10450 2    50   ~ 0
 BOOT
@@
 	5950 10450 6250 10450
 NoConn ~ 3600 10750
-NoConn ~ 4650 10750
-NoConn ~ 4800 10750
-Text Label 8750 9450 2    50   ~ 0
-GND
-$Comp
-L elements:Резистор_0,065Вт R16
-U 1 1 614557AC
-P 7425 9250
-F 0 "R16" H 7425 9125 60  0000 C CNN
-F 1 "Резистор_0,065Вт" H 7425 9100 60  0001 C CNN
-F 2 "N_RLC:Резистор_SMD_0603_0,065_Вт" H 7425 9250 60  0001 C CNN
-F 3 "" H 7425 9250 60  0001 C CNN
-F 4 "R101" H 7425 9250 50  0001 C CNN "УГО"
-F 5 "240 Ом" H 7425 9400 50  0000 C CNN "INFO"
-	1    7425 9250
-	-1   0    0    1
-$EndComp
-Wire Wire Line
-	5950 9550 6900 9550
-Wire Wire Line
-	6900 9550 6900 9250
-NoConn ~ 5950 9700
-Text Label 6750 9850 2    50   ~ 0
-LED.GREEN
-Text Label 6750 9550 2    50   ~ 0
-LED.RED
+Text Label 6750 9700 0    50   ~ 0
+LED
 $Comp
 L elements:Клеммник_х3 XS2
@@
 L elements:Резистор_0,065Вт R17
 U 1 1 61468C4F
-P 7425 9850
-F 0 "R17" H 7425 9725 60  0000 C CNN
-F 1 "Резистор_0,065Вт" H 7425 9700 60  0001 C CNN
-F 2 "N_RLC:Резистор_SMD_0603_0,065_Вт" H 7425 9850 60  0001 C CNN
-F 3 "" H 7425 9850 60  0001 C CNN
-F 4 "R101" H 7425 9850 50  0001 C CNN "УГО"
-F 5 "240 Ом" H 7425 10000 50  0000 C CNN "INFO"
-	1    7425 9850
+P 7275 9700
+F 0 "R17" H 7275 9575 60  0000 C CNN
+F 1 "Резистор_0,065Вт" H 7275 9550 60  0001 C CNN
+F 2 "N_RLC:Резистор_SMD_0603_0,065_Вт" H 7275 9700 60  0001 C CNN
+F 3 "" H 7275 9700 60  0001 C CNN
+F 4 "R101" H 7275 9700 50  0001 C CNN "УГО"
+F 5 "240 Ом" H 7275 9850 50  0000 C CNN "INFO"
+	1    7275 9700
 	-1   0    0    1
 $EndComp
-Wire Wire Line
-	5950 9850 7125 9850
-Wire Wire Line
-	6900 9250 7125 9250
-Wire Wire Line
-	7725 9250 8000 9250
-Wire Wire Line
-	7725 9850 7875 9850
-Wire Wire Line
-	7875 9850 7875 9450
-Wire Wire Line
-	7875 9450 8000 9450
-Wire Wire Line
-	8300 9250 8500 9250
-Wire Wire Line
-	8500 9250 8500 9450
-Wire Wire Line
-	8300 9450 8500 9450
-Wire Wire Line
-	8750 9450 8500 9450
-Connection ~ 8500 9450
 $Comp
 L elements:Резистор_0,065Вт R4
@@
 Wire Wire Line
 	11250 3500 11925 3500
-Text Label 1750 9400 0    50   ~ 0
+Text Label 6750 10300 2    50   ~ 0
 AN.BAT.MEASURE
-Text Label 1750 9100 0    50   ~ 0
+Text Label 5625 11000 2    50   ~ 0
 AN.2V5.REF
-NoConn ~ 2500 9250
+Wire Wire Line
+	4800 10750 4800 11000
+Wire Wire Line
+	4800 11000 5625 11000
+NoConn ~ 4650 10750
+NoConn ~ 2500 10300
+Wire Wire Line
+	6750 10300 5950 10300
+Wire Wire Line
+	5950 10000 6750 10000
+$Comp
+L BIG_schemes:Светодиод HL1
+U 1 1 61662DE6
+P 7750 9700
+F 0 "HL1" H 7725 10125 138 0000 L CNB
+F 1 "Светодиод" H 7850 9900 50  0001 C CNN
+F 2 "N_VD_HL:Светодиод_SMD_IEC_0603" H 8025 9700 50  0001 C CNN
+F 3 "" H 8025 9700 50  0001 C CNN
+F 4 "2.730" H 7850 10000 50  0001 C CNN "SYMBOL"
+	1    7750 9700
+	1    0    0    -1
+$EndComp
+Wire Wire Line
+	7575 9700 7750 9700
+Wire Wire Line
+	8450 9700 8750 9700
+Text Label 8750 9700 2    50   ~ 0
+GND
+Wire Wire Line
+	5950 9700 6975 9700
+Wire Wire Line
+	5950 9850 6750 9850
+Text Label 6750 9850 2    50   ~ 0
+SELF.TURN
+$Comp
+L elements:LOGO D1
+U 1 1 616EF452
+P 10000 7500
+F 0 "D1" H 9925 7700 50  0001 C CNN
+F 1 "LOGO" H 9900 7500 50  0000 L CNN
+F 2 "N_ICO:ni_10x10" H 10000 7500 50  0001 C CNN
+F 3 "" H 10000 7500 50  0001 C CNN
+	1    10000 7500
+	1    0    0    -1
+$EndComp
+$Comp
+L elements:LOGO D2
+U 1 1 616EF826
+P 10500 7500
+F 0 "D2" H 10425 7700 50  0001 C CNN
+F 1 "LOGO" H 10400 7500 50  0000 L CNN
+F 2 "N_ICO:VLAD_10x10" H 10500 7500 50  0001 C CNN
+F 3 "" H 10500 7500 50  0001 C CNN
+	1    10500 7500
+	1    0    0    -1
+$EndComp
 $EndSCHEMATC

Commit message: добавлена кнопка воот, перенесен Ain, начато BT arduino
Parts:
- added K2: Кнопка_KLS7-TS5401-1.35-250-T, N_X:Кнопка_KLS7-TS5401, symbol elements_2020:Кнопка_KLS7-TS5401-1.35-250-T
Connections:
- net AN.2V5.REF: now also A1.12 (IO27); no longer A1.24 (IO2)
- net BOOT: now also K2.2
- net GND: now also K2.4
- no-connect marks 3 -> 4
Changed lines of the file:
@@
 Text Label 6750 10300 2    50   ~ 0
 AN.BAT.MEASURE
-Text Label 5625 11000 2    50   ~ 0
+Text Label 2000 10150 0    50   ~ 0
 AN.2V5.REF
-Wire Wire Line
-	4800 10750 4800 11000
-Wire Wire Line
-	4800 11000 5625 11000
 NoConn ~ 4650 10750
 NoConn ~ 2500 10300
@@
 	1    0    0    -1
 $EndComp
+Wire Wire Line
+	2500 10150 2000 10150
+NoConn ~ 4800 10750
+$Comp
+L elements_2020:Кнопка_KLS7-TS5401-1.35-250-T K2
+U 1 1 61673D90
+P 9050 7150
+F 0 "K2" V 9250 7350 50  0000 R CNN
+F 1 "Кнопка_KLS7-TS5401-1.35-250-T" V 9004 7100 50  0001 R CNN
+F 2 "N_X:Кнопка_KLS7-TS5401" H 9050 7175 50  0001 C CNN
+F 3 "" H 9050 7175 50  0001 C CNN
+	1    9050 7150
+	0    -1   -1   0
+$EndComp
+Text Label 8750 6750 2    50   ~ 0
+BOOT
+Text Label 9050 6750 0    50   ~ 0
+GND
+Wire Wire Line
+	9050 6750 9050 7000
+Wire Wire Line
+	8750 6750 8750 7000
 $EndSCHEMATC
